Commit message: fix: fix  wrong package name in donner launch

File: donner_sensor_kit_description/urdf/sensor_kit.xacro (robot description, xacro)
@@ -14,4 +14,7 @@
       <child link="${sensor_kit_base_link}"/>
     </joint>
+    <!-- <link name="${sensor_kit_base_link}">
+      <origin rpy="0 0 0" xyz="0.84 0.38 0"/>
+    </link> -->
     <link name="${sensor_kit_base_link}">
       <origin rpy="0 0 0" xyz="0 0 0"/>

Commit message: chore: add FP_POI in urdf

File: donner_sensor_kit_description/urdf/sensor_kit.xacro (robot description, xacro)
@@ -55,5 +55,5 @@
     <!-- gnss -->
     <!-- <xacro:imu_macro name="gnss" parent="sensor_kit_base_link" namespace="" x="${calibration['sensor_kit_base_link']['gnss_link']['x']}" y="${calibration['sensor_kit_base_link']['gnss_link']['y']}" z="${calibration['sensor_kit_base_link']['gnss_link']['z']}" roll="${calibration['sensor_kit_base_link']['gnss_link']['roll']}" pitch="${calibration['sensor_kit_base_link']['gnss_link']['pitch']}" yaw="${calibration['sensor_kit_base_link']['gnss_link']['yaw']}" fps="100" /> -->
-    <!-- <xacro:imu_macro name="FP_POI" parent="sensor_kit_base_link" namespace="" x="${calibration['sensor_kit_base_link']['FP_POI']['x']}" y="${calibration['sensor_kit_base_link']['FP_POI']['y']}" z="${calibration['sensor_kit_base_link']['FP_POI']['z']}" roll="${calibration['sensor_kit_base_link']['FP_POI']['roll']}" pitch="${calibration['sensor_kit_base_link']['FP_POI']['pitch']}" yaw="${calibration['sensor_kit_base_link']['FP_POI']['yaw']}" fps="100" /> -->
+    <xacro:imu_macro name="FP_POI" parent="sensor_kit_base_link" namespace="" x="${calibration['sensor_kit_base_link']['FP_POI']['x']}" y="${calibration['sensor_kit_base_link']['FP_POI']['y']}" z="${calibration['sensor_kit_base_link']['FP_POI']['z']}" roll="${calibration['sensor_kit_base_link']['FP_POI']['roll']}" pitch="${calibration['sensor_kit_base_link']['FP_POI']['pitch']}" yaw="${calibration['sensor_kit_base_link']['FP_POI']['yaw']}" fps="100" />
     <!-- imu -->
     <xacro:imu_macro name="vn100" parent="sensor_kit_base_link" namespace="" x="${calibration['sensor_kit_base_link']['vn100']['x']}" y="${calibration['sensor_kit_base_link']['vn100']['y']}" z="${calibration['sensor_kit_base_link']['vn100']['z']}" roll="${calibration['sensor_kit_base_link']['vn100']['roll']}" pitch="${calibration['sensor_kit_base_link']['vn100']['pitch']}" yaw="${calibration['sensor_kit_base_link']['vn100']['yaw']}" fps="100" />

File: donner_sensor_kit_description/urdf/sensors.xacro (robot description, xacro)
@@ -1,28 +1,18 @@
 <?xml version="1.0"?>
-<robot name="vehicle" xmlns:xacro="http://ros.org/wiki/xacro">
+<robot name="vehicle"
+  xmlns:xacro="http://ros.org/wiki/xacro">
   <xacro:arg name="config_dir" default="$(find donner_sensor_kit_description)/config"/>
   <xacro:property name="calibration" value="${xacro.load_yaml('$(arg config_dir)/sensors_calibration.yaml')}"/>
   <!-- sensor kit -->
   <xacro:include filename="sensor_kit.xacro"/>
-  <xacro:sensor_kit_macro
-    parent="base_link"
-    x="${calibration['base_link']['sensor_kit_base_link']['x']}"
-    y="${calibration['base_link']['sensor_kit_base_link']['y']}"
-    z="${calibration['base_link']['sensor_kit_base_link']['z']}"
-    roll="${calibration['base_link']['sensor_kit_base_link']['roll']}"
-    pitch="${calibration['base_link']['sensor_kit_base_link']['pitch']}"
-    yaw="${calibration['base_link']['sensor_kit_base_link']['yaw']}"
-  />
+  <xacro:sensor_kit_macro parent="base_link" x="${calibration['base_link']['sensor_kit_base_link']['x']}" y="${calibration['base_link']['sensor_kit_base_link']['y']}" z="${calibration['base_link']['sensor_kit_base_link']['z']}" roll="${calibration['base_link']['sensor_kit_base_link']['roll']}" pitch="${calibration['base_link']['sensor_kit_base_link']['pitch']}" yaw="${calibration['base_link']['sensor_kit_base_link']['yaw']}" />
   <!-- embedded sensors -->
   <!-- <xacro:include filename="$(find velodyne_description)/urdf/VLP-16.urdf.xacro"/>
   <xacro:VLP-16 parent="base_link" name="velodyne_rear" topic="velodyne_rear/velodyne_points" hz="10" samples="220" gpu="false">
-    <origin
-      xyz="${calibration['base_link']['velodyne_rear_base_link']['x']}
+    <origin xyz="${calibration['base_link']['velodyne_rear_base_link']['x']}
            ${calibration['base_link']['velodyne_rear_base_link']['y']}
-           ${calibration['base_link']['velodyne_rear_base_link']['z']}"
-      rpy="${calibration['base_link']['velodyne_rear_base_link']['roll']}
+           ${calibration['base_link']['velodyne_rear_base_link']['z']}" rpy="${calibration['base_link']['velodyne_rear_base_link']['roll']}
            ${calibration['base_link']['velodyne_rear_base_link']['pitch']}
-           ${calibration['base_link']['velodyne_rear_base_link']['yaw']}"
-    />
+           ${calibration['base_link']['velodyne_rear_base_link']['yaw']}" />
   </xacro:VLP-16> -->
 </robot>
