Commit message: add velodyne

File: athena_sensor_kit_description/urdf/sensor_kit.xacro (robot description, xacro)
@@ -41,4 +41,13 @@
              ${calibration['sensor_kit_base_link']['velodyne_right_base_link']['yaw']}" />
     </xacro:VLP-16> -->
+    <xacro:VLP-16 parent="sensor_kit_base_link" name="velodyne_top" topic="/points_raw" hz="10" samples="220" gpu="$(arg gpu)">
+      <origin
+             xyz="${calibration['sensor_kit_base_link']['velodyne_top_base_link']['x']}
+             ${calibration['sensor_kit_base_link']['velodyne_top_base_link']['y']}
+             ${calibration['sensor_kit_base_link']['velodyne_top_base_link']['z']}"
+             rpy="${calibration['sensor_kit_base_link']['velodyne_top_base_link']['roll']}
+             ${calibration['sensor_kit_base_link']['velodyne_top_base_link']['pitch']}
+             ${calibration['sensor_kit_base_link']['velodyne_top_base_link']['yaw']}" />
+    </xacro:VLP-16>
     <!-- camera -->
     <!-- <xacro:monocular_camera_macro name="traffic_light_right_camera/camera" parent="sensor_kit_base_link" namespace="" x="${calibration['sensor_kit_base_link']['traffic_light_right_camera/camera_link']['x']}" y="${calibration['sensor_kit_base_link']['traffic_light_right_camera/camera_link']['y']}" z="${calibration['sensor_kit_base_link']['traffic_light_right_camera/camera_link']['z']}" roll="${calibration['sensor_kit_base_link']['traffic_light_right_camera/camera_link']['roll']}" pitch="${calibration['sensor_kit_base_link']['traffic_light_right_camera/camera_link']['pitch']}" yaw="${calibration['sensor_kit_base_link']['traffic_light_right_camera/camera_link']['yaw']}" fps="30" width="800" height="400" fov="1.3" />

Commit message: feat: teleware

File: athena_sensor_kit_description/urdf/sensor_kit.xacro (robot description, xacro)
@@ -42,11 +42,16 @@
     </xacro:VLP-16> -->
     <xacro:VLP-16 parent="sensor_kit_base_link" name="velodyne_top" topic="/points_raw" hz="10" samples="220" gpu="$(arg gpu)">
-      <origin
-             xyz="${calibration['sensor_kit_base_link']['velodyne_top_base_link']['x']}
+      <origin xyz="${calibration['sensor_kit_base_link']['velodyne_top_base_link']['x']}
              ${calibration['sensor_kit_base_link']['velodyne_top_base_link']['y']}
-             ${calibration['sensor_kit_base_link']['velodyne_top_base_link']['z']}"
-             rpy="${calibration['sensor_kit_base_link']['velodyne_top_base_link']['roll']}
+             ${calibration['sensor_kit_base_link']['velodyne_top_base_link']['z']}" rpy="${calibration['sensor_kit_base_link']['velodyne_top_base_link']['roll']}
              ${calibration['sensor_kit_base_link']['velodyne_top_base_link']['pitch']}
              ${calibration['sensor_kit_base_link']['velodyne_top_base_link']['yaw']}" />
+    </xacro:VLP-16>
+    <xacro:VLP-16 parent="sensor_kit_base_link" name="hesai_top" topic="/points_raw" hz="10" samples="220" gpu="$(arg gpu)">
+      <origin xyz="${calibration['sensor_kit_base_link']['hesai_top_base_link']['x']}
+             ${calibration['sensor_kit_base_link']['hesai_top_base_link']['y']}
+             ${calibration['sensor_kit_base_link']['hesai_top_base_link']['z']}" rpy="${calibration['sensor_kit_base_link']['hesai_top_base_link']['roll']}
+             ${calibration['sensor_kit_base_link']['hesai_top_base_link']['pitch']}
+             ${calibration['sensor_kit_base_link']['hesai_top_base_link']['yaw']}" />
     </xacro:VLP-16>
     <!-- camera -->

Commit message: test: past test

File: athena_sensor_kit_description/urdf/sensor_kit.xacro (robot description, xacro)
@@ -48,5 +48,5 @@
              ${calibration['sensor_kit_base_link']['velodyne_top_base_link']['yaw']}" />
     </xacro:VLP-16> -->
-    <xacro:VLP-16 parent="sensor_kit_base_link" name="hesai_top" topic="/points_raw" hz="10" samples="220" gpu="$(arg gpu)">
+    <!-- <xacro:VLP-16 parent="sensor_kit_base_link" name="hesai_top" topic="/points_raw" hz="10" samples="220" gpu="$(arg gpu)">
       <origin xyz="${calibration['sensor_kit_base_link']['hesai_top_base_link']['x']}
              ${calibration['sensor_kit_base_link']['hesai_top_base_link']['y']}
@@ -54,4 +54,11 @@
              ${calibration['sensor_kit_base_link']['hesai_top_base_link']['pitch']}
              ${calibration['sensor_kit_base_link']['hesai_top_base_link']['yaw']}" />
+    </xacro:VLP-16> -->
+    <xacro:VLP-16 parent="sensor_kit_base_link" name="helios_top" topic="/points_raw" hz="10" samples="220" gpu="$(arg gpu)">
+      <origin xyz="${calibration['sensor_kit_base_link']['rs_helios_top']['x']}
+             ${calibration['sensor_kit_base_link']['rs_helios_top']['y']}
+             ${calibration['sensor_kit_base_link']['rs_helios_top']['z']}" rpy="${calibration['sensor_kit_base_link']['rs_helios_top']['roll']}
+             ${calibration['sensor_kit_base_link']['rs_helios_top']['pitch']}
+             ${calibration['sensor_kit_base_link']['rs_helios_top']['yaw']}" />
     </xacro:VLP-16>
     <!-- camera -->

Commit message: feat: fuse helios32 and m1

File: athena_sensor_kit_description/urdf/sensor_kit.xacro (robot description, xacro)
@@ -55,10 +55,19 @@
              ${calibration['sensor_kit_base_link']['hesai_top_base_link']['yaw']}" />
     </xacro:VLP-16> -->
-    <xacro:VLP-16 parent="sensor_kit_base_link" name="helios_top" topic="/points_raw" hz="10" samples="220" gpu="$(arg gpu)">
+    <xacro:VLP-16 parent="sensor_kit_base_link" name="rs_helios_top" topic="/points_raw" hz="10" samples="220" gpu="$(arg gpu)">
       <origin xyz="${calibration['sensor_kit_base_link']['rs_helios_top']['x']}
              ${calibration['sensor_kit_base_link']['rs_helios_top']['y']}
-             ${calibration['sensor_kit_base_link']['rs_helios_top']['z']}" rpy="${calibration['sensor_kit_base_link']['rs_helios_top']['roll']}
+             ${calibration['sensor_kit_base_link']['rs_helios_top']['z']}"
+             rpy="${calibration['sensor_kit_base_link']['rs_helios_top']['roll']}
              ${calibration['sensor_kit_base_link']['rs_helios_top']['pitch']}
              ${calibration['sensor_kit_base_link']['rs_helios_top']['yaw']}" />
+    </xacro:VLP-16>
+    <xacro:VLP-16 parent="sensor_kit_base_link" name="rs_m1_right" topic="/points_raw" hz="10" samples="220" gpu="$(arg gpu)">
+      <origin xyz="${calibration['sensor_kit_base_link']['rs_m1_right']['x']}
+             ${calibration['sensor_kit_base_link']['rs_m1_right']['y']}
+             ${calibration['sensor_kit_base_link']['rs_m1_right']['z']}"
+             rpy="${calibration['sensor_kit_base_link']['rs_m1_right']['roll']}
+             ${calibration['sensor_kit_base_link']['rs_m1_right']['pitch']}
+             ${calibration['sensor_kit_base_link']['rs_m1_right']['yaw']}" />
     </xacro:VLP-16>
     <!-- camera -->
